Commit message: Can pass num_robots and randomness seed into nodes through launchfile

File: nuturtle_description/urdf/common_properties.xacro (robot description, xacro)
@@ -32,4 +32,13 @@
     <color rgba="0.8 0.0 0.0 1.0"/>
   </material>
+  <material name="cyan">
+    <color rgba="0.0 0.8 0.8 1.0"/>
+  </material>
+  <material name="magenta">
+    <color rgba="0.8 0.0 0.8 1.0"/>
+  </material>
+  <material name="yellow">
+    <color rgba="0.8 0.8 0.0 1.0"/>
+  </material>
   <material name="white">
     <color rgba="1.0 1.0 1.0 1.0"/>
